File: Hardware/DM50.kicad_pcb (KiCad board)
At the start: 2 copper layers, 43 parts, among them J1 ST-LINK, J2 USB_C_Receptacle_USB2.0_14P, Q1 MMBT3904, SW16 R, U1 EA_DOGL128X-6, U2 STM32U535CBT6, U3 W25Q32JVSS, U4 ADP2108AUJ-3.3

Commit message: Shematic changes
Other:
- board outline added: 71 x 138 mm
Changed lines of the file:
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@@
 			(type default)
 		)
-		(layer "Margin")
+		(layer "Edge.Cuts")
 	)
 	(gr_line
@@
 			(type default)
 		)
-		(layer "Margin")
+		(layer "Edge.Cuts")
 	)
 	(gr_line
@@
 			(type default)
 		)
-		(layer "Margin")
+		(layer "Edge.Cuts")
 	)
 	(gr_line
@@
 			(type default)
 		)
-		(layer "Margin")
+		(layer "Edge.Cuts")
 	)
 	(gr_line
@@
 			(type default)
 		)
-		(layer "User.1")
+		(layer "F.Fab")
 	)
 	(gr_line
@@
 			(type default)
 		)
-		(layer "User.1")
+		(layer "F.Fab")
 	)
 	(gr_line
@@
 			(type default)
 		)
-		(layer "User.1")
+		(layer "F.Fab")
 	)
 	(gr_line
@@
 			(type default)
 		)
-		(layer "User.1")
+		(layer "F.Fab")
 	)
 )
