File: Hardware/DM50.kicad_sch (KiCad schematic)
At the start: 67 parts

Commit message: electronic design advances
Parts:
- removed C? (x2): 10u, Capacitor_SMD:C_0603_1608Metric, symbol Device:C
- removed C?: 100n, Capacitor_SMD:C_0402_1005Metric, symbol Device:C
- removed C? (x2): 47pF, symbol Device:C
- removed C?: 100nF, symbol Device:C
- removed F?: 100mA, Fuse:Fuse_1206_3216Metric, symbol Device:Fuse
- removed FB?: 100 @ 100MHz, Inductor_SMD:L_0805_2012Metric, symbol Device:Ferrite_Bead
- removed J?: ST-LINK, symbol Connector_Generic:Conn_01x04
- removed J?: ARM 10pin, Connector_PinHeader_1.27mm:PinHeader_2x05_P1.27mm_Vertical, symbol Connector_Generic:Conn_02x05_Odd_Even
- removed J?: USB_B_Micro, 10118193-0001LF:101181930001LF, symbol Connector:USB_B_Micro
- removed R? (x2): 10k, symbol Device:R
- removed SW?: "Reset", symbol Switch:SW_Push
- removed U?: STM32L476VGT6, Package_QFP:LQFP-100_14x14mm_P0.5mm, symbol MCU_ST_STM32L4:STM32L476VGTx
- removed U?: USBLC6-2SC6, Package_TO_SOT_SMD:SOT-23-6, symbol Power_Protection:USBLC6-2SC6
- removed U?: XC6206P332MR, Package_TO_SOT_SMD:SOT-23, symbol Regulator_Linear:XC6206PxxxMR
- removed Y?: 32768Hz, symbol Device:Crystal
- added BT1: 2xAAA (1.5V), Battery:BatteryHolder_Keystone_2468_2xAAA, symbol Device:Battery_Cell
- added BZ1: Buzzer, Connector:JWT_A3963_1x02_P3.96mm_Vertical, symbol Device:Buzzer
- added C1: 100nF, Capacitor_SMD:C_0603_1608Metric, symbol Device:C
- added C10, C2, C3, C4, C5, C6, C7, C8, C9: 1uF, Capacitor_SMD:C_0603_1608Metric, symbol Device:C
- added C11, C12: 8pF, Capacitor_SMD:C_0603_1608Metric, symbol Device:C
- added C13: 2.2uF, Capacitor_SMD:C_0603_1608Metric, symbol Device:C
- added C14: 104, Capacitor_SMD:C_0603_1608Metric, symbol Device:C
- added C15: 4.7 uF, Capacitor_SMD:C_0603_1608Metric, symbol Device:C
- added C16: 10 uF, Capacitor_SMD:C_0603_1608Metric, symbol Device:C
- added D1: LED (RED), LED_SMD:LED_0603_1608Metric, symbol Device:LED
- added D2: BAT54C, Package_TO_SOT_SMD:SOT-23, symbol Diode:BAT54C
- added J1: ST-LINK, Connector_PinHeader_1.00mm:PinHeader_1x05_P1.00mm_Vertical, symbol Connector_Generic:Conn_01x05
- added J2: USB_C_Receptacle_USB2.0_14P, Connector_USB:USB_C_Receptacle_GCT_USB4105-xx-A_16P_TopMnt_Horizontal, symbol Connector:USB_C_Receptacle_USB2.0_14P
- added L1: 1uH, Inductor_SMD:L_0805_2012Metric_Pad1.15x1.40mm_HandSolder, symbol Device:L
- added Q1: MMBT3904, Package_TO_SOT_SMD:SOT-23, symbol Transistor_BJT:MMBT3904
- added R1: 10k, Resistor_SMD:R_0603_1608Metric, symbol Device:R
- added R2: 4.7K, Resistor_SMD:R_0603_1608Metric, symbol Device:R
- added R3, R4: 10K, Resistor_SMD:R_0603_1608Metric, symbol Device:R
- added R5, R6: R, Resistor_SMD:R_0603_1608Metric, symbol Device:R
- added R7, R8, R9: 5.1K, Resistor_SMD:R_0603_1608Metric, symbol Device:R
- added SW7: "Reset", symbol Switch:SW_Push
- added U1: EA_DOGL128X-6, Display:EA_DOGL128-6, symbol Display_Graphic:EA_DOGL128X-6
- added U2: STM32U535CBT6, Package_QFP:LQFP-48_7x7mm_P0.5mm, symbol MCU_ST_STM32U5:STM32U535CBTx
- added U3: W25Q32JVSS, Package_SO:SOIC-8_5.23x5.23mm_P1.27mm, symbol Memory_Flash:W25Q32JVSS
- added U4: ADP2108AUJ-3.3, Package_TO_SOT_SMD:TSOT-23-5, symbol Regulator_Switching:ADP2108AUJ-3.3
- added Y1: 25MHz 9PF, symbol Device:Crystal
- C17, C18, C19, C20, C21: renamed from C?; footprint (none) -> Capacitor_SMD:C_0603_1608Metric
- SW10: renamed from SW?; value TRI -> SQR
- SW11: renamed from SW?; value ln -> LOG
- SW12: renamed from SW?; value e^x -> LN
- SW13: renamed from SW?; value x^2 -> XEQ
- SW16: renamed from SW?; value Rv -> R; footprint (none) -> Resistor_SMD:R_0603_1608Metric
- SW17: renamed from SW?; value CC -> SIN
- SW18: renamed from SW?; value f -> COS
- SW19: renamed from SW?; value g -> TAN
- SW25: renamed from SW?; value <- -> DEL
- SW26: renamed from SW?; value / -> UP
- SW30: renamed from SW?; value XEQ -> /
- SW31: renamed from SW?; value x -> DOWN
- SW35: renamed from SW?; value UP -> x
- SW36: renamed from SW?; value - -> OPT
- SW40: renamed from SW?; value DOWN -> -
- SW41: renamed from SW?; value + -> ON
- SW45: renamed from SW?; value EXIT -> +
- SW8: renamed from SW?; value 1/x -> E+
- SW9: renamed from SW?; value y^x -> 1/x
- gave numbers to parts that had none: 25
Connections:
- net GND: now also BT1.2 (-), C1.2, C11.2, C12.2, C13.2, C14.1, C15.2, C16.2, C2.2, C3.2, C4.2, C6.2, C7.2, C9.1, D1.1 (K), J1.1 (Pin_1), J2.A1 (GND), J2.A12 (GND), J2.B1 (GND), J2.B12 (GND), J2.S1 (SHIELD), Q1.2 (E), R4.1, R8.2, R9.2, SW7.1, U1.26 (VSS), U1.33 (VSS), U2.23 (VSS), U2.35 (VSS), U2.47 (VSS), U2.8 (VSSA), U3.4 (GND), U4.2 (GND)
- net NRST: now also C1.1, J1.5 (Pin_5), R1.2, SW7.2, U2.7 (NRST)
- net SWCLK: now also J1.3 (Pin_3), U2.37 (PA14)
- net SWDIO: now also J1.4 (Pin_4), U2.34 (PA13)
- net +BATT renamed 3.3V
- net 3.3V: now also SW41.1, BZ1.1 (+), C16.1, L1.2, R1.1, R2.2, R5.1, U1.34 (VDD2), U1.35 (VDD), U2.1 (VBAT), U2.24 (VDD), U2.36 (VDD), U2.48 (VDD), U2.9 (VDDA), U3.3 (IO2), U3.7 (IO3), U3.8 (VCC), U4.4 (FB)
- net kh1 renamed ROW08
- net ROW08: now also U2.28 (PB15); no longer SW41.2
- net kh2 renamed ROW07
- net ROW07: now also U2.27 (PB14)
- net kh3 renamed ROW06
- net ROW06: now also U2.26 (PB13)
- net kh4 renamed ROW05
- net ROW05: now also U2.25 (PB12)
- net kh5 renamed ROW04
- net ROW04: now also U2.21 (PB10)
- net kh6 renamed ROW03
- net ROW03: now also U2.46 (PB9)
- net kh7 renamed ROW02
- net ROW02: now also U2.45 (PB8)
- net kh8 renamed ROW01
- net ROW01: now also U2.42 (PB6)
- net kv1 renamed COL01
- net COL01: now also U2.18 (PB0); no longer SW41.1
- net kv2 renamed COL02
- net COL02: now also U2.19 (PB1)
- net kv3 renamed COL03
- net COL03: now also U2.30 (PA9)
- net kv4 renamed COL04
- net COL04: now also U2.20 (PB2)
- net kv5 renamed COL05
- net COL05: now also U2.29 (PA8)
- net kv6 renamed COL06
- net COL06: now also U2.38 (PA15)
- new net: C2.1, U1.21 (V0)
- new net: C3.1, U1.22 (V1)
- new net: C4.1, U1.23 (V2)
- new net: C6.1, U1.24 (V3)
- new net: C7.1, U1.25 (V4)
- new net: C10.1, U1.27 (CAP2N)
- new net: C10.2, U1.28 (CAP2P)
- new net: C5.1, U1.29 (CAP1P)
- new net: C5.2, C8.2, U1.30 (CAP1N)
- new net: C8.1, U1.31 (CAP3P)
- new net: C9.2, U1.32 (VOUT)
- new net: BZ1.2 (-), Q1.3 (C), R5.2
- new net: R2.1, U3.1 (~{CS})
- new net: C13.1, U2.22 (VCAP)
- new net: C11.1, U2.5 (PH0), Y1.1
- new net: C12.1, U2.6 (PH1), Y1.2
- new net: Q1.1 (B), R6.2
- new net: C15.1, D2.3, U4.1 (Vin)
- new net: BT1.1 (+), D2.1
- new net: D2.2, J2.A4 (VBUS), J2.A9 (VBUS), J2.B4 (VBUS), J2.B9 (VBUS)
- new net: R3.2, R4.2, SW41.2
- new net: L1.1, U4.5 (SW)
- new net: J2.B5 (CC2), R9.1
- new net: J2.A5 (CC1), R8.1
- new net: D1.2 (A), R7.2
- new net BUZZER: R6.1, U2.40 (PB4)
- new net DISP_A0: U1.38 (A0), U2.12 (PA2)
- new net DISP_CS1B: U1.40 (~{CS1B}), U2.13 (PA3)
- new net DISP_RST: U1.39 (~{RST}), U2.14 (PA4)
- new net DISP_SCL: U1.37 (SCL), U2.10 (PA0)
- new net DISP_SI: U1.36 (SI), U2.11 (PA1)
- new net LED01: R7.1, U2.41 (PB5)
- new net POWER_ON: U2.4 (PC15), U4.3 (EN)
- new net SPI_MISO: U2.16 (PA6), U3.2 (DO(IO1))
- new net SPI_MOSI: U2.17 (PA7), U3.5 (DI(IO0))
- new net SPI_SCK: U2.15 (PA5), U3.6 (CLK)
- new net SWO: J1.2 (Pin_2), U2.39 (PB3)
- new net USB_DM (D-): J2.A7 (D-), J2.B7 (D-), U2.32 (PA11)
- new net USB_DP (D+): J2.A6 (D+), J2.B6 (D+), U2.33 (PA12)
- new net WAKEUP01: C14.2, R3.1, U2.2 (PC13)
- no-connect marks 19 -> 10
Other:
- note added: "Display Visions EA DOGL128L-6 (L is reflective, without leds) FSTN 128X64 ST7565R 320uA https://www.digikey.es/es/products/detail/display-visions/EA-DOGL128L-6/4896695 https://www.lcd-module.com/eng/pdf/grafik/dogl128-6e.pdf Regulators: DM42 LD3985, OpenRPNCalc TPS61222TCK, PUSH Panasonic EVQQ2B01W"
- note added: "VREFINT"
- note removed: "3V3 Regulator"
- note removed: "Limit USB host-side cap to <= 10uF to ensure we're not hitting maximum in-rush current when device is attached. See: http://www.ti.com/lit/an/slyt118/slyt118.pdf"
- note removed: "NRST cap not strictly necessary but protects against parasitic resets."
- note removed: "Not reverse polarity protected,however since only power source is via USB connector, we can hope that the polarity will be correct."
- note removed: "STM32 USB requires 3V3."
- note removed: "SWD Connector"
- note removed: "USB Connector and ESD Protection"
- note removed: "max. 200mA @ 3V3"
- moved on the sheet: C17, C18, C19, C20, C21, SW1, SW10, SW11, SW12, SW13, SW14, SW15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

Commit message: Shematic changes
Parts:
- removed C14: 104, Capacitor_SMD:C_0603_1608Metric, symbol Device:C
- removed J1: ST-LINK, Connector_PinHeader_1.00mm:PinHeader_1x05_P1.00mm_Vertical, symbol Connector_Generic:Conn_01x05
- removed R4: 10K, Resistor_SMD:R_0603_1608Metric, symbol Device:R
- removed SW7: "Reset", symbol Switch:SW_Push
- added J3: ST-LINK, symbol Connector_Generic:Conn_01x05
- added R10: 100K, Resistor_SMD:R_0603_1608Metric, symbol Device:R
- added SW46: SW_RESET, symbol Switch:SW_Push
- added U5: USBLC6-2SC6, Package_TO_SOT_SMD:SOT-23-6, symbol Power_Protection:USBLC6-2SC6
- C11, C12: value 8pF -> 22pF
- Y1: value 25MHz 9PF -> HC/49US 8MHz
Connections:
- net 3.3V: now also R3.1; no longer SW41.1
- net COL01: now also SW41.1
- net GND: now also J3.1 (Pin_1), R10.2, SW46.1, U5.2 (GND)
- net NRST: now also J3.5 (Pin_5)
- net POWER_ON: no longer U4.3 (EN)
- net ROW01: now also U2.26 (PB13); no longer U2.42 (PB6)
- net ROW06: no longer U2.26 (PB13)
- net ROW08: no longer SW42.2, SW43.2, SW44.2, SW45.2
- net SWCLK: now also J3.3 (Pin_3)
- net SWDIO: now also J3.2 (Pin_2)
- net SWO: now also J3.4 (Pin_4)
- net USB_DM (D-): now also U5.6 (I/O1); no longer J2.A7 (D-), J2.B7 (D-)
- net USB_DP (D+): now also U5.4 (I/O2); no longer J2.A6 (D+), J2.B6 (D+)
- net at R3.2: now also U4.3 (EN), SW46.2; no longer SW41.2
- net WAKEUP01 renamed ROW06/WAKEUP
- net ROW06/WAKEUP: no longer R3.1
- new net: J2.A7 (D-), J2.B7 (D-), U5.1 (I/O1)
- new net: J2.A6 (D+), J2.B6 (D+), U5.3 (I/O2)
- new net ROW08/WAKEUP: R10.1, SW41.2, SW42.2, SW43.2, SW44.2, SW45.2
- new net VBUS: U5.5 (VBUS)
Other:
- note added: "R WakeUp"
- moved on the sheet: BT1, C1, C11, C12, C15, C16, C17, C18, C19, C20, C21, D2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
