File: hardware/DM50 copia.kicad_pcb (KiCad board)
At the start: 2 copper layers, 70 x 138 mm, 93 parts, among them J1 ST-LINK, J2 USB_C_Receptacle_USB2.0_14P, Q1 MMBT3904, SW1 F1, SW10 LOG, SW11 LN, SW12 XEQ, SW13 STO, SW14 RCL, SW15 R, SW16 SIN, SW17 COS, SW18 TAN, SW19 ENTER, SW2 F2, SW20 ENTER, SW21 x<>y, SW22 +/-, SW23 E, SW24 DEL, SW25 UP, SW26 7, SW27 8, SW28 9, SW29 /, SW3 F3, SW30 DOWN, SW31 4, SW32 5, SW33 6, SW34 x, SW35 OPT, SW36 1, SW37 2, SW38 3, SW39 -, SW4 F4, SW40 ON, SW41 0, SW42 ., SW43 =, SW44 +, SW45 SW_RESET, SW5 F5, SW6 F6, SW7 E+, SW8 1/x, SW9 SQR, U1 EA_DOGL128X-6, U2 STM32U535CBT6, U3 AT25SF641, U4 USBLC6-2SC6, U5 ADP2108AUJ-3.3, Y1 HSE 16MHz

Commit message: pcb changes
Parts:
- BT1, BT2: footprint DM50:dm50-batAAA -> DM50:dm50-batAA
- moved C10 5.94 mm to (68.5, 53.0)
- moved C11 5.94 mm to (68.5, 57.0)
- moved C12 5.94 mm to (68.5, 65.0)
- moved C13 5.94 mm to (68.5, 59.0)
- moved C14 5.94 mm to (68.5, 51.0)
- moved C17 5.94 mm to (68.5, 67.0)
- moved C18 5.94 mm to (68.5, 49.0)
- moved R1 5.94 mm to (68.5, 55.0)
- moved R3 5.94 mm to (68.5, 61.0)
- moved R6 5.94 mm to (68.5, 63.0)
- moved BZ1 5.50 mm to (93.9, 45.0)
- moved C19 4.03 mm to (86.8, 73.0)
- moved C20 4.03 mm to (81.2, 69.8)
- moved C21 4.03 mm to (81.2, 67.8)
- moved L1 4.03 mm to (90.6, 70.3)
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Routing:
- net GND: track 312.5 -> 0.00 mm, vias 2 -> 0
- net ROW08/WAKEUP: track 205.2 -> 12.5 mm, vias 0 -> 5
- net COL02: track 176.2 -> 0.00 mm, vias 4 -> 0
- net BOOT0: track 192.1 -> 33.7 mm, vias 2 -> 5
- net 3.3V: track 146.4 -> 0.00 mm, vias 7 -> 0
- net ROW07: track 175.9 -> 33.7 mm, vias 2 -> 5
- net COL05: track 117.1 -> 0.00 mm, vias 1 -> 0
- net ROW03: track 150.2 -> 33.7 mm, vias 2 -> 5
- net COL03: track 114.2 -> 0.00 mm, vias 1 -> 0
- net ROW05: track 146.7 -> 33.7 mm, vias 2 -> 5
- net COL04: track 108.2 -> 0.00 mm, vias 1 -> 0
- net ROW04: track 132.8 -> 33.7 mm, vias 4 -> 5
- net COL06: track 91.7 -> 0.00 mm, vias 1 -> 0
- net ROW02: track 114.5 -> 40.5 mm, vias 2 -> 6
- net NRST: track 65.1 -> 0.00 mm, vias 4 -> 0
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Other:
- outline, holes or cut-outs redrawn
