File: hardware/DM50.kicad_sch (KiCad schematic)
At the start: 92 parts, among them J1 ST-LINK, J2 USB_C_Receptacle_USB2.0_14P, Q1 MMBT3904, SW1 F1, SW10 SQR, SW11 LOG, SW12 LN, SW13 XEQ, SW14 STO, SW15 RCL, SW16 R, SW17 SIN, SW18 COS, SW19 TAN, SW2 F2, SW20 ENTER, SW21 ENTER, SW22 x<>y, SW23 +/-, SW24 E, SW25 DEL, SW26 UP, SW27 7, SW28 8, SW29 9, SW3 F3, SW30 /, SW31 DOWN, SW32 4, SW33 5, SW34 6, SW35 x, SW36 OPT, SW37 1, SW38 2, SW39 3, SW4 F4, SW40 -, SW41 ON, SW42 0, SW43 ., SW44 R/S, SW45 +, SW46 SW_RESET, SW5 F5, SW6 F6, SW8 E+, SW9 1/x, U1 EA_DOGL128X-6, U2 STM32U535CBT6, U3 AT25SF641, U4 ADP2108AUJ-3.3, U5 USBLC6-2SC6, Y1 HSE 16MHz

Commit message: update 3d render
Parts:
- J1: footprint (none) -> Connector_JST:JST_XH_B5B-XH-AM_1x05_P2.50mm_Vertical
- SW1, SW2, SW3, SW4, SW5, SW6: footprint (none) -> DM50:dm50-button
- SW10: renamed from SW11; footprint (none) -> DM50:dm50-button
- SW11: renamed from SW12; footprint (none) -> DM50:dm50-button
- SW12: renamed from SW13; footprint (none) -> DM50:dm50-button
- SW13: renamed from SW14; footprint (none) -> DM50:dm50-button
- SW14: renamed from SW15; footprint (none) -> DM50:dm50-button
- SW15: renamed from SW16; footprint Resistor_SMD:R_0603_1608Metric -> DM50:dm50-button
- SW16: renamed from SW17; footprint (none) -> DM50:dm50-button
- SW17: renamed from SW18; footprint (none) -> DM50:dm50-button
- SW18: renamed from SW19; footprint (none) -> DM50:dm50-button
- SW19: renamed from SW20; footprint (none) -> DM50:dm50-button
- SW20: renamed from SW21; footprint (none) -> DM50:dm50-button
- SW21: renamed from SW22; footprint (none) -> DM50:dm50-button
- SW22: renamed from SW23; footprint (none) -> DM50:dm50-button
- SW23: renamed from SW24; footprint (none) -> DM50:dm50-button
- SW24: renamed from SW25; footprint (none) -> DM50:dm50-button
- SW25: renamed from SW26; footprint (none) -> DM50:dm50-button
- SW26: renamed from SW27; footprint (none) -> DM50:dm50-button
- SW27: renamed from SW28; footprint (none) -> DM50:dm50-button
- SW28: renamed from SW29; footprint (none) -> DM50:dm50-button
- SW29: renamed from SW30; footprint (none) -> DM50:dm50-button
- SW30: renamed from SW31; footprint (none) -> DM50:dm50-button
- SW31: renamed from SW32; footprint (none) -> DM50:dm50-button
- SW32: renamed from SW33; footprint (none) -> DM50:dm50-button
- SW33: renamed from SW34; footprint (none) -> DM50:dm50-button
- SW34: renamed from SW35; footprint (none) -> DM50:dm50-button
- SW35: renamed from SW36; footprint (none) -> DM50:dm50-button
- SW36: renamed from SW37; footprint (none) -> DM50:dm50-button
- SW37: renamed from SW38; footprint (none) -> DM50:dm50-button
- SW38: renamed from SW39; footprint (none) -> DM50:dm50-button
- SW39: renamed from SW40; footprint (none) -> DM50:dm50-button
- SW40: renamed from SW41; footprint (none) -> DM50:dm50-button
- SW41: renamed from SW42; footprint (none) -> DM50:dm50-button
- SW42: renamed from SW43; footprint (none) -> DM50:dm50-button
- SW43: renamed from SW44; value R/S -> =; footprint (none) -> DM50:dm50-button
- SW44: renamed from SW45; footprint (none) -> DM50:dm50-button
- SW45: renamed from SW46; footprint (none) -> Button_Switch_SMD:SW_SPST_TL3342
- SW7: renamed from SW8; footprint (none) -> DM50:dm50-button
- SW8: renamed from SW9; footprint (none) -> DM50:dm50-button
- SW9: renamed from SW10; footprint (none) -> DM50:dm50-button
- U3: footprint Package_SO:SOIC-8_5.23x5.23mm_P1.27mm -> Package_SO:SOIC-8_3.9x4.9mm_P1.27mm
- Y1: footprint (none) -> Crystal:Crystal_SMD_0603-2Pin_6.0x3.5mm
- renumbered C2 to C1, C1 to C10, C12 to C11, C13 to C12, C11 to C13, C17 to C14, C18 to C15, C19 to C16, C20 to C17, C21 to C18, C16 to C19, C3 to C2, C14 to C20, C15 to C21, C4 to C3, C5 to C4, C6 to C5, C7 to C6, C8 to C7, C9 to C8, C10 to C9, R8 to R10, R9 to R11, R3 to R12, R7 to R2, R2 to R3, R10 to R4, R4 to R5, R12 to R6, R11 to R7, R5 to R8, R6 to R9, U5 to U4, U4 to U5

Commit message: pcb changes
Parts:
- added BT2: AA, DM50:dm50-batAA, symbol Device:Battery_Cell
- BT1: value 2xAAA (1.5V) -> AA; footprint Battery:BatteryHolder_Keystone_2468_2xAAA -> DM50:dm50-batAA
- renumbered C21 to C20, C20 to C21
Connections:
- net GND: now also BT2.2 (-); no longer BT1.2 (-)
- net VBAT: no longer D2.1
- new net: BT1.2 (-), BT2.1 (+)
Other:
- note added: "Display Visions EA DOGL128L-6 (L is reflective, without leds) https://www.digikey.es/es/products/detail/display-visions/EA-DOGL128L-6/4896695 Regulators LD3985, TPS61222TCK, Battery: https://www.digikey.es/es/products/detail/keystone-electronics/54/2254090"
- note removed: "Display Visions EA DOGL128L-6 (L is reflective, without leds) FSTN 128X64 ST7565R 320uA https://www.digikey.es/es/products/detail/display-visions/EA-DOGL128L-6/4896695 https://www.lcd-module.com/eng/pdf/grafik/dogl128-6e.pdf Regulators: DM42 LD3985, OpenRPNCalc TPS61222TCK, PUSH Panasonic EVQQ2B01W"
- moved on the sheet: BT1, C19, C20, D2, L1, R12, SW45, U5

Commit message: changes
Parts:
- BZ1: footprint Connector:JWT_A3963_1x02_P3.96mm_Vertical -> DM50:Buzzer
- J1: footprint Connector_JST:JST_XH_B5B-XH-AM_1x05_P2.50mm_Vertical -> DM50:JST_CON_SMD
- U1: footprint Display:EA_DOGL128-6 -> DM50:EA_DOGL128-6
Changed lines of the file:
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@@
 			)
 		)
-		(property "Footprint" "Display:EA_DOGL128-6"
+		(property "Footprint" "DM50:EA_DOGL128-6"
 			(at 245.11 41.91 0)
 			(effects
@@
 			)
 		)
-		(property "Footprint" "Connector:JWT_A3963_1x02_P3.96mm_Vertical"
+		(property "Footprint" "DM50:Buzzer"
 			(at 269.875 142.24 90)
 			(effects
@@
 			)
 		)
-		(property "Footprint" "Connector_JST:JST_XH_B5B-XH-AM_1x05_P2.50mm_Vertical"
+		(property "Footprint" "DM50:JST_CON_SMD"
 			(at 186.69 92.71 0)
 			(effects

Commit message: pcb changes
Parts:
- BT1, BT2: footprint DM50:dm50-batAA -> DM50:dm50-batAAA
Changed lines of the file:
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@@
 			)
 		)
-		(property "Footprint" "DM50:dm50-batAA"
+		(property "Footprint" "DM50:dm50-batAAA"
 			(at 82.55 181.356 90)
 			(effects
@@
 			)
 		)
-		(property "Footprint" "DM50:dm50-batAA"
+		(property "Footprint" "DM50:dm50-batAAA"
 			(at 82.55 188.976 90)
 			(effects

Commit message: pcb changes
Parts:
- C11, C13: value 22pF -> 10pF
- R8: value R -> 100K
- R9: value R -> 10K
Other:
- note added: "BOOT"
Changed lines of the file:
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@@
 		)
 	)
+	(text "BOOT"
+		(exclude_from_sim no)
+		(at 37.084 91.186 0)
+		(effects
+			(font
+				(size 0.508 0.508)
+			)
+		)
+	)
 	(global_label "VCAP1"
 		(shape input)
@@
 			)
 		)
-		(property "Value" "R"
+		(property "Value" "100K"
 			(at 261.874 147.32 90)
 			(effects
@@
 			)
 		)
-		(property "Value" "22pF"
+		(property "Value" "10pF"
 			(at 53.848 141.986 90)
 			(effects
@@
 			)
 		)
-		(property "Value" "22pF"
+		(property "Value" "10pF"
 			(at 54.102 128.524 90)
 			(effects
@@
 			)
 		)
-		(property "Value" "R"
-			(at 251.968 151.638 90)
+		(property "Value" "10K"
+			(at 252.73 151.384 90)
 			(effects
 				(font

Commit message: pcb changes
Connections:
- net VBAT: now also D2.1
Other:
- moved on the sheet: BT1, BT2
Changed lines of the file:
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@@
 	)
 	(junction
+		(at 82.55 179.07)
+		(diameter 0)
+		(color 0 0 0 0)
+	)
+	(junction
 		(at 39.37 55.88)
 		(diameter 0)
@@
 	)
 	(junction
+		(at 82.55 163.83)
+		(diameter 0)
+		(color 0 0 0 0)
+	)
+	(junction
 		(at 243.84 20.32)
 		(diameter 0)
@@
 	)
 	(junction
-		(at 82.55 163.83)
-		(diameter 0)
-		(color 0 0 0 0)
-	)
-	(junction
 		(at 35.56 82.55)
 		(diameter 0)
@@
 		)
 	)
-	(wire
-		(pts
-			(xy 81.28 177.8) (xy 82.55 177.8)
-		)
-		(stroke
-			(width 0)
-			(type default)
-		)
-	)
 	(polyline
 		(pts
@@
 	(wire
 		(pts
+			(xy 81.28 179.07) (xy 82.55 179.07)
+		)
+		(stroke
+			(width 0)
+			(type default)
+		)
+	)
+	(wire
+		(pts
 			(xy 26.67 113.03) (xy 35.56 113.03)
 		)
@@
 	(symbol
 		(lib_id "power:+BATT")
-		(at 81.28 177.8 90)
+		(at 81.28 179.07 90)
 		(unit 1)
 		(exclude_from_sim no)
@@
 		(dnp no)
 		(property "Reference" "#PWR027"
-			(at 85.09 177.8 0)
+			(at 85.09 179.07 0)
 			(effects
 				(font
@@
 		)
 		(property "Value" "VBAT"
-			(at 76.454 177.8 90)
+			(at 76.454 179.07 90)
 			(effects
 				(font
@@
 		)
 		(property "Footprint" ""
-			(at 81.28 177.8 0)
+			(at 81.28 179.07 0)
 			(effects
 				(font
@@
 		)
 		(property "Datasheet" ""
-			(at 81.28 177.8 0)
+			(at 81.28 179.07 0)
 			(effects
 				(font
@@
 		)
 		(property "Description" ""
-			(at 81.28 177.8 0)
+			(at 81.28 179.07 0)
 			(effects
 				(font
@@
 	(symbol
 		(lib_id "power:GND")
-		(at 82.55 193.04 0)
+		(at 82.55 194.31 0)
 		(unit 1)
 		(exclude_from_sim no)
@@
 		(fields_autoplaced yes)
 		(property "Reference" "#PWR035"
-			(at 82.55 199.39 0)
+			(at 82.55 200.66 0)
 			(effects
 				(font
@@
 		)
 		(property "Value" "GND"
-			(at 82.55 198.12 0)
+			(at 82.55 199.39 0)
 			(effects
 				(font
@@
 		)
 		(property "Footprint" ""
-			(at 82.55 193.04 0)
+			(at 82.55 194.31 0)
 			(effects
 				(font
@@
 		)
 		(property "Datasheet" ""
-			(at 82.55 193.04 0)
+			(at 82.55 194.31 0)
 			(effects
 				(font
@@
 		)
 		(property "Description" ""
-			(at 82.55 193.04 0)
+			(at 82.55 194.31 0)
 			(effects
 				(font
@@
 	(symbol
 		(lib_id "Device:Battery_Cell")
-		(at 82.55 182.88 0)
+		(at 82.55 184.15 0)
 		(unit 1)
 		(exclude_from_sim no)
@@
 		(dnp no)
 		(property "Reference" "BT1"
-			(at 77.978 180.086 0)
+			(at 77.978 181.356 0)
 			(effects
 				(font
@@
 		)
 		(property "Value" "AA"
-			(at 77.978 182.88 0)
+			(at 77.978 184.15 0)
 			(effects
 				(font
@@
 		)
 		(property "Footprint" "DM50:dm50-batAAA"
-			(at 82.55 181.356 90)
+			(at 82.55 182.626 90)
 			(effects
 				(font
@@
 		)
 		(property "Datasheet" "~"
-			(at 82.55 181.356 90)
+			(at 82.55 182.626 90)
 			(effects
 				(font
@@
 		)
 		(property "Description" "Single-cell battery"
-			(at 82.55 182.88 0)
+			(at 82.55 184.15 0)
 			(effects
 				(font
@@
 	(symbol
 		(lib_id "Device:Battery_Cell")
-		(at 82.55 190.5 0)
+		(at 82.55 191.77 0)
 		(unit 1)
 		(exclude_from_sim no)
@@
 		(dnp no)
 		(property "Reference" "BT2"
-			(at 78.486 187.452 0)
+			(at 78.486 188.722 0)
 			(effects
 				(font
@@
 		)
 		(property "Value" "AA"
-			(at 78.232 190.5 0)
+			(at 78.232 191.77 0)
 			(effects
 				(font
@@
 		)
 		(property "Footprint" "DM50:dm50-batAAA"
-			(at 82.55 188.976 90)
+			(at 82.55 190.246 90)
 			(effects
 				(font
@@
 		)
 		(property "Datasheet" "~"
-			(at 82.55 188.976 90)
+			(at 82.55 190.246 90)
 			(effects
 				(font
@@
 		)
 		(property "Description" "Single-cell battery"
-			(at 82.55 190.5 0)
+			(at 82.55 191.77 0)
 			(effects
 				(font

Commit message: pcb changes
Parts:
- removed R4: 10K, Resistor_SMD:R_0603_1608Metric, symbol Device:R
- removed R7: 100K, Resistor_SMD:R_0603_1608Metric, symbol Device:R
- added R1: 100k, Resistor_SMD:R_0603_1608Metric, symbol Device:R
- added R12: 10K, Resistor_SMD:R_0603_1608Metric, symbol Device:R
- added SW10: CST, DM50:dm50-button, symbol Switch:SW_Push_45deg
- added SW11: VAR, DM50:dm50-button, symbol Switch:SW_Push_45deg
- added SW12: U, DM50:dm50-button, symbol Switch:SW_Push_45deg
- added SW13: NXT, DM50:dm50-button, symbol Switch:SW_Push_45deg
- added SW8: MTH, DM50:dm50-button, symbol Switch:SW_Push_45deg
- added SW9: PRG, DM50:dm50-button, symbol Switch:SW_Push_45deg
- SW14: renamed from SW7; value E+ -> '
- SW15: renamed from SW8; value 1/x -> STO
- SW16: renamed from SW9; value SQR -> EVAL
- SW17: renamed from SW10; value LOG -> L
- SW18: renamed from SW11; value LN -> D
- SW19: renamed from SW12; value XEQ -> R
- SW20: renamed from SW13; value STO -> SIN
- SW21: renamed from SW14; value RCL -> COS
- SW22: renamed from SW15; value R -> TAN
- SW23: renamed from SW16; value SIN -> SQR
- SW24: renamed from SW17; value COS -> y^x
- SW25: renamed from SW18; value TAN -> 1/x
- SW28: renamed from SW21; value x<>y -> +/-
- SW29: renamed from SW22; value +/- -> EEX
- SW30: renamed from SW23; value E -> DEL
- SW31: renamed from SW24; value DEL -> BACK
- SW32: renamed from SW25; value UP -> ALPHA
- SW37: renamed from SW30; value DOWN -> OPT1
- SW42: renamed from SW45; value SW_RESET -> RESET
- SW43: renamed from SW35; value OPT -> OPT2
- SW51: renamed from SW43; value = -> SPC
- renumbered R11 to R10, R12 to R11, R1 to R2, R2 to R3, R3 to R4, R8 to R7, R9 to R8, R10 to R9, SW1 to SW2, SW19 to SW26, SW20 to SW27, SW2 to SW3, SW26 to SW33, SW27 to SW34, SW28 to SW35, SW29 to SW36, SW31 to SW38, SW32 to SW39, SW3 to SW4, SW33 to SW40, SW34 to SW41, SW36 to SW44, SW37 to SW45, SW38 to SW46, SW39 to SW47, SW40 to SW48, SW41 to SW49, SW4 to SW5, SW42 to SW50, SW44 to SW52, SW5 to SW6, SW6 to SW7
Connections:
- net POWER_ON is gone; now on net ROW08: U2.4 (PC15)
- net 3.3V: now also R12.1
- net BOOT0: now also U2.27 (PB14), R1.1
- net BUZZER: now also U2.40 (PB4); no longer U2.42 (PB6)
- net COL01: now also SW8.1
- net COL02: now also U2.12 (PA2), R12.2, SW9.1; no longer U2.40 (PB4)
- net COL03: now also U2.14 (PA4), SW10.1; no longer U2.30 (PA9)
- net COL04: now also U2.15 (PA5), SW11.1; no longer U2.20 (PB2)
- net COL05: now also U2.20 (PB2), SW12.1; no longer U2.29 (PA8)
- net COL06: now also U2.21 (PB10), SW13.1; no longer U2.38 (PA15)
- net DISP_A0: now also U2.43 (PB7); no longer U2.14 (PA4)
- net DISP_CS1B: now also U2.46 (PB9); no longer U2.15 (PA5)
- net DISP_RST: now also U2.45 (PB8); no longer U2.31 (PA10)
- net DISP_SCL: now also U2.42 (PB6); no longer U2.12 (PA2)
- net DISP_SI: now also U2.38 (PA15); no longer U2.43 (PB7)
- net GND: now also SW42.2, R1.2; no longer SW42.1
- net LED01: now also U2.25 (PB12); no longer U2.41 (PB5)
- net NRST: now also J1.4 (Pin_4), SW42.1; no longer J1.5 (Pin_5)
- net ROW01: now also U2.41 (PB5); no longer U2.26 (PB13)
- net ROW02: now also U2.31 (PA10), SW10.2, SW11.2, SW12.2, SW13.2, SW8.2, SW9.2; no longer SW14.2, SW15.2, SW16.2, SW17.2, SW18.2, SW19.2, U2.45 (PB8)
- net ROW03: now also SW14.2, SW15.2, SW16.2, SW17.2, SW18.2, SW19.2, U2.30 (PA9); no longer SW20.2, SW21.2, SW22.2, SW23.2, SW24.2, SW25.2, U2.46 (PB9)
- net ROW04: now also SW20.2, SW21.2, SW22.2, SW23.2, SW24.2, SW25.2, U2.29 (PA8); no longer SW26.2, SW27.2, SW28.2, SW29.2, SW30.2, SW31.2, U2.21 (PB10)
- net ROW05: now also SW26.2, SW27.2, SW28.2, SW29.2, SW30.2, SW31.2, U2.26 (PB13); no longer SW32.2, SW33.2, SW34.2, SW35.2, SW36.2, U2.25 (PB12)
- net ROW08: now also SW43.2, SW44.2, SW45.2, SW46.2, SW47.2; no longer U2.28 (PB15)
- net SWD_SWO: now also J1.5 (Pin_5); no longer J1.4 (Pin_4)
- net at R11.2, U5.3 (EN): no longer SW42.2
- net ROW06/WAKEUP renamed ROW06
- net ROW06: now also SW32.2, SW33.2, SW34.2, SW35.2, SW36.2
- removed net ROW07: SW43.2, SW44.2, SW45.2, SW46.2, SW47.2, U2.27 (PB14)
- net ROW08/WAKEUP renamed ROW09/WAKEUP
- net ROW09/WAKEUP: now also U2.28 (PB15)
Other:
- note added: "KEY COL02 - ROW07"
- moved on the sheet: C10, C19, C21, J1, L1, R11, R2, SW14, SW15, SW16, SW17, SW18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

Commit message: pcb and rendeer
Parts:
- SW14: value ' -> quote
Changed lines of the file:
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@@
 			)
 		)
-		(property "Value" "'"
+		(property "Value" "quote"
 			(at 25.654 48.514 0)
 			(effects
