File: hardware/DM50.kicad_pcb (KiCad board)
At the start: 2 copper layers, 70 x 138 mm, 93 parts, among them J1 ST-LINK, J2 USB_C_Receptacle_USB2.0_14P, Q1 MMBT3904, SW1 F1, SW10 LOG, SW11 LN, SW12 XEQ, SW13 STO, SW14 RCL, SW15 R, SW16 SIN, SW17 COS, SW18 TAN, SW19 ENTER, SW2 F2, SW20 ENTER, SW21 x<>y, SW22 +/-, SW23 E, SW24 DEL, SW25 UP, SW26 7, SW27 8, SW28 9, SW29 /, SW3 F3, SW30 DOWN, SW31 4, SW32 5, SW33 6, SW34 x, SW35 OPT, SW36 1, SW37 2, SW38 3, SW39 -, SW4 F4, SW40 ON, SW41 0, SW42 ., SW43 =, SW44 +, SW45 SW_RESET, SW5 F5, SW6 F6, SW7 E+, SW8 1/x, SW9 SQR, U1 EA_DOGL128X-6, U2 STM32U535CBT6, U3 AT25SF641, U4 USBLC6-2SC6, U5 ADP2108AUJ-3.3, Y1 HSE 16MHz

Commit message: pcb changes
Routing:
- net ROW01: track 101.1 -> 116.4 mm
- net ROW03: track 135.3 -> 149.4 mm
- net ROW08/WAKEUP: track 160.5 -> 169.7 mm
- net ROW05: track 142.9 -> 149.5 mm
- net BOOT0: track 177.0 -> 182.3 mm
- net ROW04: track 130.4 -> 133.6 mm
- net COL02: track 127.0 -> 124.1 mm
- net ROW02: track 118.9 -> 121.8 mm
- net COL04: track 107.6 -> 109.9 mm
- net Net-(U1-V3): track 3.96 -> 6.03 mm
- net Net-(U1-CAP3P): track 3.98 -> 6.03 mm
- net Net-(U1-V0): track 3.98 -> 6.03 mm
- net Net-(U1-V2): track 4.00 -> 6.04 mm
- net Net-(U1-V1): track 4.00 -> 6.04 mm
- net GND: track 308.9 -> 310.9 mm
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
Commit message: pcb changes
Parts:
- removed SW1: F1, DM50:dm50-button
- added SW2: F1, DM50:dm50-button, F.Cu at (55.5, 88.0)
- added SW20: SIN, DM50:dm50-button, F.Cu at (55.5, 121.0)
- added SW21: COS, DM50:dm50-button, F.Cu at (67.0, 121.0)
- added SW22: TAN, DM50:dm50-button, F.Cu at (78.5, 121.0)
- added SW23: SQR, DM50:dm50-button, F.Cu at (90.0, 121.0)
- added SW24: y^x, DM50:dm50-button, F.Cu at (101.5, 121.0)
- added SW25: 1/x, DM50:dm50-button, F.Cu at (113.0, 121.0)
- R1: value 10k -> 100k
- R11: value 5.1K -> 10K
- R2: value 5.1K -> 10k
- R3: value 1M -> 5.1K
- R4: value 10K -> 1M
- R8: value 100K -> 10K
- R9: value 10K -> 5.1K
- SW10: renamed from SW9; value SQR -> CST
- SW11: renamed from SW10; value LOG -> VAR
- SW12: renamed from SW11; value LN -> U
- SW13: renamed from SW12; value XEQ -> NXT
- SW14: renamed from SW13; value STO -> '
- SW15: renamed from SW14; value RCL -> STO
- SW16: renamed from SW15; value R -> EVAL
- SW17: renamed from SW16; value SIN -> L
- SW18: renamed from SW17; value COS -> D
- SW19: renamed from SW18; value TAN -> R
- SW28: renamed from SW21; value x<>y -> +/-
- SW29: renamed from SW22; value +/- -> EEX
- SW30: renamed from SW23; value E -> DEL
- SW31: renamed from SW24; value DEL -> BACK
- SW32: renamed from SW25; value UP -> ALPHA
- SW37: renamed from SW30; value DOWN -> OPT1
- SW42: value . -> RESET; footprint DM50:dm50-button -> Button_Switch_SMD:SW_SPST_TL3342; moved to B.Cu
- SW43: renamed from SW35; value OPT -> OPT2
- SW50: renamed from SW45; value SW_RESET -> .; footprint Button_Switch_SMD:SW_SPST_TL3342 -> DM50:dm50-button; moved to F.Cu
- SW51: renamed from SW43; value = -> SPC
- SW8: renamed from SW7; value E+ -> MTH
- SW9: renamed from SW8; value 1/x -> PRG
- moved SW50 123.5 mm to (84.5, 176.0), turned to 0 degrees
- moved SW42 113.1 mm to (55.3, 55.8), turned to -90 degrees
- moved R3 29.1 mm to (101.4, 73.6), turned to -90 degrees
- moved R11 24.8 mm to (90.1, 68.4), turned to -90 degrees
- moved R5 24.4 mm to (96.8, 73.5), turned to 90 degrees
- moved R1 23.5 mm to (85.7, 73.5)
- moved R9 23.4 mm to (109.5, 56.8), turned to -90 degrees
- moved C12 21.7 mm to (93.6, 62.8), turned to 0 degrees
- moved R6 21.1 mm to (93.6, 64.7), turned to 180 degrees
- moved C10 18.2 mm to (75.7, 36.8), turned to 0 degrees
- moved R2 17.7 mm to (72.3, 36.8)
- moved R4 13.2 mm to (93.6, 60.8), turned to 0 degrees
- moved R12 11.8 mm to (75.1, 73.6)
- moved SW26 11.0 mm to (55.5, 132.0)
- moved SW27 11.0 mm to (67.0, 132.0)
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- renumbered SW19 to SW26, SW20 to SW27, SW2 to SW3, SW26 to SW33, SW27 to SW34, SW28 to SW35, SW29 to SW36, SW31 to SW38, SW32 to SW39, SW3 to SW4, SW33 to SW40, SW34 to SW41, SW36 to SW44, SW37 to SW45, SW38 to SW46, SW39 to SW47, SW40 to SW48, SW41 to SW49, SW4 to SW5, SW44 to SW52, SW5 to SW6, SW6 to SW7
Connections:
- J1 pad 4: SWD_SWO -> NRST
- J1 pad 5: NRST -> SWD_SWO
- R1 pad 1: 3.3V -> BOOT0
- R1 pad 2: NRST -> GND
- R10 pad 1: Net-(J2-CC1) -> Net-(J2-CC2)
- R11 pad 1: Net-(J2-CC2) -> Net-(U5-Vin)
- R11 pad 2: GND -> Net-(U5-EN)
- R12 pad 1: Net-(U5-Vin) -> 3.3V
- R12 pad 2: Net-(U5-EN) -> COL02
- R2 pad 1: LED01 -> 3.3V
- R2 pad 2: Net-(D1-A) -> NRST
- R3 pad 1: VBAT_SNS -> LED01
- R3 pad 2: VBAT -> Net-(D1-A)
- R4 pad 1: COL02 -> VBAT_SNS
- R4 pad 2: 3.3V -> VBAT
- R5 pad 1: ROW08/WAKEUP -> ROW09/WAKEUP
- R7 pad 1: GND -> 3.3V
- R7 pad 2: BOOT0 -> Net-(BZ1--)
- R8 pad 1: 3.3V -> BUZZER
- R8 pad 2: Net-(BZ1--) -> Net-(Q1-B)
- R9 pad 1: BUZZER -> Net-(J2-CC1)
- R9 pad 2: Net-(Q1-B) -> GND
- SW26 pad 2: ROW04 -> ROW05
- SW27 pad 2: ROW04 -> ROW05
- SW28 pad 2: ROW04 -> ROW05
- SW29 pad 2: ROW04 -> ROW05
- SW30 pad 2: ROW04 -> ROW05
- SW31 pad 2: ROW04 -> ROW05
- SW32 pad 2: ROW05 -> ROW06
- SW33 pad 2: ROW05 -> ROW06
- SW34 pad 2: ROW05 -> ROW06
- SW35 pad 2: ROW05 -> ROW06
- SW36 pad 2: ROW05 -> ROW06
- SW42 pad 1: COL03 -> NRST
- SW42 pad 2: ROW08/WAKEUP -> GND
- SW43 pad 2: ROW07 -> ROW08
- SW44 pad 2: ROW07 -> ROW08
- SW45 pad 2: ROW07 -> ROW08
- SW46 pad 2: ROW07 -> ROW08
- SW47 pad 2: ROW07 -> ROW08
- SW48 pad 2: ROW08/WAKEUP -> ROW09/WAKEUP
- SW49 pad 2: ROW08/WAKEUP -> ROW09/WAKEUP
- SW50 pad 1: GND -> COL03
- SW50 pad 2: Net-(U5-EN) -> ROW09/WAKEUP
- SW51 pad 2: ROW08/WAKEUP -> ROW09/WAKEUP
- SW52 pad 2: ROW08/WAKEUP -> ROW09/WAKEUP
- U2 pad 12: DISP_SCL -> COL02
- U2 pad 14: DISP_A0 -> COL03
- U2 pad 15: DISP_CS1B -> COL04
- U2 pad 2: ROW06/WAKEUP -> ROW06
- U2 pad 20: COL04 -> COL05
- U2 pad 21: ROW04 -> COL06
- U2 pad 25: ROW05 -> LED01
- U2 pad 26: ROW01 -> ROW05
- U2 pad 27: ROW07 -> BOOT0
- U2 pad 28: ROW08 -> ROW09/WAKEUP
- U2 pad 29: COL05 -> ROW04
- U2 pad 30: COL03 -> ROW03
- U2 pad 31: DISP_RST -> ROW02
- U2 pad 38: COL06 -> DISP_SI
- U2 pad 4: POWER_ON -> ROW08
- U2 pad 40: COL02 -> BUZZER
- U2 pad 41: LED01 -> ROW01
- U2 pad 42: BUZZER -> DISP_SCL
- U2 pad 43: DISP_SI -> DISP_A0
- U2 pad 45: ROW02 -> DISP_RST
- U2 pad 46: ROW03 -> DISP_CS1B
Routing:
- net ROW09/WAKEUP: track 0.00 -> 181.5 mm, vias 0 -> 2
- net ROW08/WAKEUP: track 169.7 -> 0.00 mm, vias 2 -> 0
- net ROW07: track 167.8 -> 0.00 mm, vias 2 -> 0
- net ROW08: track 0.00 -> 153.7 mm, vias 0 -> 2
- net ROW06: track 0.00 -> 130.1 mm, vias 0 -> 2
- net GND: track 310.9 -> 222.6 mm, vias 2 -> 1
- net Net-(U5-EN): track 56.9 -> 1.87 mm, vias 1 -> 0
- net Net-(D1-A): track 64.9 -> 12.6 mm, vias 2 -> 0
- net SWD_SWDIO: track 49.9 -> 0.00 mm, vias 1 -> 0
- net 3.3V: track 126.5 -> 78.4 mm, vias 5 -> 0
- net Net-(BT1--): track 53.4 -> 12.0 mm, vias 1 -> 0
- net VBAT: track 55.7 -> 15.1 mm
- net ROW03: track 149.4 -> 110.9 mm
- net DISP_RST: track 64.5 -> 29.9 mm, vias 1 -> 0
- net DISP_A0: track 61.9 -> 27.9 mm, vias 2 -> 0
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- removed copper zone on F.Cu, net GND
Other:
- board size 70 x 138 mm -> 70 x 149.5 mm
- board text removed: "USBC"

Commit message: pcb and rendeer
Parts:
- SW14: value ' -> quote
- moved R12 11.5 mm to (76.8, 62.2), turned to 180 degrees
- moved R5 7.41 mm to (102.2, 68.5)
- moved R1 3.20 mm to (83.0, 71.8), turned to 0 degrees
Routing:
- net Net-(BT1--): track 12.0 -> 90.0 mm
- net 3.3V: track 78.4 -> 145.1 mm, vias 0 -> 6
- net BOOT0: track 151.6 -> 212.8 mm, vias 2 -> 5
- net ROW01: track 86.0 -> 140.6 mm, vias 2 -> 3
- net ROW02: track 89.1 -> 141.7 mm, vias 2 -> 3
- net ROW04: track 110.9 -> 161.6 mm, vias 2 -> 3
- net ROW03: track 110.9 -> 160.3 mm, vias 2 -> 3
- net ROW06: track 130.1 -> 171.6 mm, vias 2 -> 4
- net COL02: track 109.5 -> 149.7 mm, vias 1 -> 2
- net COL01: track 94.3 -> 133.7 mm, vias 1 -> 2
- net ROW08: track 153.7 -> 191.3 mm, vias 2 -> 3
- net ROW05: track 122.6 -> 159.3 mm, vias 2 -> 5
- net COL06: track 53.9 -> 87.1 mm
- net ROW09/WAKEUP: track 181.5 -> 214.6 mm, vias 2 -> 4
- net SWD_SWDIO: track 0.00 -> 22.7 mm, vias 0 -> 1
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- added copper zone on B.Cu, net GND
- added copper zone on F.Cu, net GND

Commit message: Update DM50.kicad_pcb
Parts:
- moved R1 3.63 mm to (86.5, 70.8), turned to 180 degrees
Routing:
- net ROW01: track 140.6 -> 147.1 mm
- net BOOT0: track 212.8 -> 206.7 mm
- net NRST: track 68.1 -> 64.4 mm
- net Net-(BT1--): track 90.0 -> 93.1 mm
- net ROW09/WAKEUP: track 214.6 -> 213.3 mm
- net VBAT_SNS: track 21.9 -> 20.8 mm
- net Net-(U4-VBUS): track 18.4 -> 17.4 mm, vias 2 -> 0
- net GND: track 231.6 -> 232.4 mm, vias 28 -> 30
- net Net-(J2-D+-PadA6): track 11.4 -> 10.6 mm

Commit message: pcb changes
Routing:
- net GND: vias 30 -> 32
Changed lines of the file:
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@@
 			(usegerberattributes yes)
 			(usegerberadvancedattributes yes)
-			(creategerberjobfile yes)
+			(creategerberjobfile no)
 			(dashed_line_dash_ratio 12.000000)
 			(dashed_line_gap_ratio 3.000000)
@@
 			(drillshape 0)
 			(scaleselection 1)
-			(outputdirectory "")
+			(outputdirectory "gerbers/")
 		)
 	)
@@
 	)
 	(via
+		(at 109.1 46.8)
+		(size 0.8)
+		(drill 0.4)
+		(layers "F.Cu" "B.Cu")
+		(free yes)
+		(net 2)
+	)
+	(via
 		(at 88.5 41)
 		(size 0.8)
@@
 		(size 0.8)
 		(drill 0.4)
+		(layers "F.Cu" "B.Cu")
+		(free yes)
+		(net 2)
+	)
+	(via
+		(at 56.5 48.4)
+		(size 0.8)
+		(drill 0.4)

Commit message: pcb changes
Routing:
- net GND: vias 32 -> 31
Other:
- outline, holes or cut-outs redrawn
- board text added: "M2x5 Flat Head"
- board text removed: "DM50 calculator r1.0 https://github.com/xavierbasc/dm50-calculator"

Commit message: pcb changes
Other:
- board text added: "1.5 AAA"
- board text removed: "1.5 AA"

Commit message: pcb changes
Parts:
- moved C12 37.7 mm to (116.0, 93.2)
- moved C8 37.7 mm to (101.5, 67.2)
- moved C9 37.7 mm to (114.2, 67.2)
- moved R2 37.7 mm to (94.7, 67.2)
- moved R4 37.7 mm to (116.0, 91.2)
- moved BZ1 37.7 mm to (111.0, 74.2)
- moved C10 37.7 mm to (98.0, 67.2)
- moved C16 37.7 mm to (99.2, 90.5)
- moved C4 37.7 mm to (109.5, 67.2)
- moved C7 37.7 mm to (106.0, 67.2)
- moved D2 37.7 mm to (126.5, 87.8)
- moved R1 37.7 mm to (108.8, 101.2)
- moved R3 37.7 mm to (123.8, 104.0)
- moved R9 37.7 mm to (131.8, 87.2)
- moved U2 37.7 mm to (105.5, 86.2)
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Routing:
- net COL02: track 149.7 -> 150.2 mm
Other:
- board size 70 x 149.5 mm -> 70 x 148.5 mm
