File: hardware/DM50.kicad_pcb (KiCad board)
At the start: 2 copper layers, 70 x 149.9 mm, 99 parts, among them J1 ST-LINK, J2 USB_C_Receptacle_USB2.0_14P, Q1 MMBT3904, SW1 PGM, SW10 CST, SW11 VAR, SW12 U, SW13 NXT, SW14 quote, SW15 STO, SW16 EVAL, SW17 L, SW18 D, SW19 R, SW2 F1, SW20 SIN, SW21 COS, SW22 TAN, SW23 SQR, SW24 y^x, SW25 1/x, SW26 ENTER, SW27 ENTER, SW28 +/-, SW29 EEX, SW3 F2, SW30 DEL, SW31 BACK, SW32 ALPHA, SW33 7, SW34 8, SW35 9, SW36 /, SW37 OPT1, SW38 4, SW39 5, SW4 F3, SW40 6, SW41 x, SW42 RESET, SW43 OPT2, SW44 1, SW45 2, SW46 3, SW47 -, SW48 ON, SW49 0, SW5 F4, SW50 ., SW51 SPC, SW52 +, SW6 F5, SW7 F6, SW8 MTH, SW9 PRG, U1 EA_DOGL128X-6, U2 STM32U535CBT6, U3 AT25SF641, U4 USBLC6-2SC6, U5 ADP2108AUJ-3.3, Y1 32768

Commit message: pcb changes
Parts:
- moved BT1 1.63 mm to (129.9, 92.8)
- moved BT2 1.63 mm to (129.9, 78.0)
- moved D2 1.45 mm to (127.0, 87.8)
Routing:
- net 3.3V: track 192.4 -> 175.4 mm, vias 10 -> 8
- net ROW07: track 138.0 -> 132.7 mm
- net ROW04: track 103.4 -> 98.2 mm
- net ROW08: track 145.2 -> 150.1 mm
- net Net-(BT1--): track 109.2 -> 113.6 mm
- net BOOT0: track 61.6 -> 58.1 mm
- net ROW06: track 127.5 -> 124.2 mm
- net GND: track 164.5 -> 162.2 mm, vias 62 -> 139
- net ROW01: track 81.7 -> 79.6 mm
- net LED01: track 25.5 -> 23.4 mm
- net COL04: track 121.9 -> 124.0 mm
- net ROW03: track 92.0 -> 90.0 mm
- net ROW05: track 102.8 -> 100.9 mm
- net VBAT: track 14.5 -> 16.2 mm
- net ROW02: track 85.9 -> 84.6 mm
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Other:
- outline, holes or cut-outs redrawn
- board text added: "M2x5"

Commit message: 3d case
Routing:
- net QUADSPI_IO0: track 8.05 -> 8.75 mm
- net 3.3V: track 175.4 -> 176.0 mm
Other:
- board size 70 x 149.9 mm -> 70 x 151 mm

Commit message: 3d changes (step files)
Parts:
- added C22: 4.7 uF, Capacitor_SMD:C_0603_1608Metric, F.Cu at (122.1, 88.0)
- added C23: 4.7 uF, Capacitor_SMD:C_0603_1608Metric, F.Cu at (116.3, 87.8)
- added D3: LED (RED), LED_SMD:LED_0603_1608Metric, F.Cu at (133.6, 116.2)
- added J3: S2B-PH-K-SLFSN, DM50:CONN_S2B-PH-K-S_JST, F.Cu at (130.1, 105.7)
- added R12: 2K, Resistor_SMD:R_0603_1608Metric, F.Cu at (121.3, 86.0)
- added R13: 1.5K, Resistor_SMD:R_0603_1608Metric, F.Cu at (134.3, 98.8)
- added U6: MCP73831-2-OT, Package_TO_SOT_SMD:SOT-23-5, F.Cu at (119.3, 88.0)
- D1: value LED (RED) -> LED (GREEN)
- R1, R2: value 10k -> 10K
- SW1: value PGM -> SW_SPST
- SW10: value CST -> BT_SMD
- SW11: value VAR -> BT_SMD
- SW12: value U -> BT_SMD
- SW13: value NXT -> BT_SMD
- SW14: value quote -> BT_SMD
- SW15: value STO -> BT_SMD
- SW16: value EVAL -> BT_SMD
- SW17: value L -> BT_SMD
- SW18: value D -> BT_SMD
- SW19: value R -> BT_SMD
- SW2: value F1 -> BT_SMD
- SW20: value SIN -> BT_SMD
- SW21: value COS -> BT_SMD
- SW22: value TAN -> BT_SMD
- SW23: value SQR -> BT_SMD
- SW24: value y^x -> BT_SMD
- SW25: value 1/x -> BT_SMD
- SW26, SW27: value ENTER -> BT_SMD
- SW28: value +/- -> BT_SMD
- SW29: value EEX -> BT_SMD
- SW3: value F2 -> BT_SMD
- SW30: value DEL -> BT_SMD
- SW31: value BACK -> BT_SMD
- SW32: value ALPHA -> BT_SMD
- SW33: value 7 -> BT_SMD
- SW34: value 8 -> BT_SMD
- SW35: value 9 -> BT_SMD
- SW36: value / -> BT_SMD
- SW37: value OPT1 -> BT_SMD
- SW38: value 4 -> BT_SMD
- SW39: value 5 -> BT_SMD
- SW4: value F3 -> BT_SMD
- SW40: value 6 -> BT_SMD
- SW41: value x -> BT_SMD
- SW42: value RESET -> SW_SPST
- SW43: value OPT2 -> BT_SMD
- SW44: value 1 -> BT_SMD
- SW45: value 2 -> BT_SMD
- SW46: value 3 -> BT_SMD
- SW47: value - -> BT_SMD
- SW48: value ON -> BT_SMD
- SW49: value 0 -> BT_SMD
- SW5: value F4 -> BT_SMD
- SW50: value . -> BT_SMD
- SW51: value SPC -> BT_SMD
- SW52: value + -> BT_SMD
- SW6: value F5 -> BT_SMD
- SW7: value F6 -> BT_SMD
- SW8: value MTH -> BT_SMD
- SW9: value PRG -> BT_SMD
Connections:
- net Net-(U4-VBUS) renamed VBUS
Routing:
- net Net-(D3-K): track 0.00 -> 44.2 mm, vias 0 -> 2
- net VBAT: track 16.2 -> 37.1 mm
- net VBUS: track 17.6 -> 37.2 mm
- net Net-(D3-A): track 0.00 -> 16.7 mm
- net GND: track 162.2 -> 165.7 mm, vias 139 -> 135
- net Net-(U6-PROG): track 0.00 -> 1.07 mm
Other:
- board text added: "+ LiPO (optional)"
- board text added: "- LiPO (optional)"

Commit message: pcb changes
Parts:
- moved R12 0.45 mm to (121.3, 85.5)
- moved C22 0.05 mm to (122.2, 88.0)
Connections:
- C20 pad 1: Net-(U5-Vin) -> VINPUT
- D2 pad 3: Net-(U5-Vin) -> VINPUT
- R11 pad 1: Net-(U5-Vin) -> VINPUT
- R4 pad 2: VBAT -> VINPUT
- U2 pad 1: 3.3V -> VBAT
- U5 pad 1: Net-(U5-Vin) -> VINPUT
Routing:
- net VINPUT: track 0.00 -> 29.4 mm
- net Net-(U5-Vin): track 23.4 -> 0.00 mm
- net VBAT: track 37.1 -> 32.8 mm
- net 3.3V: track 176.0 -> 174.9 mm
- net GND: track 165.7 -> 166.7 mm, vias 135 -> 134

Commit message: pcb changes
Parts:
- removed J3: S2B-PH-K-SLFSN, DM50:CONN_S2B-PH-K-S_JST
- added J4: Conn_01x04, DM50:CONN_S2B-ZR-SM4A-TFLFSN_JST, F.Cu at (129.0, 103.1)
Routing:
- net VBAT: track 32.8 -> 53.0 mm, vias 0 -> 2
- net GND: track 166.7 -> 170.7 mm
- net 3.3V: track 174.9 -> 176.7 mm
- net NRST: track 57.1 -> 58.7 mm
- net ROW01: track 79.6 -> 80.5 mm

Commit message: LiPO CONNECTOR
Parts:
- added D4: schottky, Diode_SMD:D_SOD-323, F.Cu at (122.8, 88.8)
- added JP1: LiPO, Jumper:SolderJumper-2_P1.3mm_Bridged_RoundedPad1.0x1.5mm, F.Cu at (123.1, 85.5)
- BT1, BT2: value AA -> AAA
- J4: value Conn_01x04 -> LiPO 3,7V; footprint DM50:CONN_S2B-ZR-SM4A-TFLFSN_JST -> DM50:CONN_S2B-PH-K-S_JST
- U6: value MCP73831-2-OT -> MCP73831
- Y1: footprint Crystal:Crystal_SMD_MicroCrystal_CM9V-T1A-2Pin_1.6x1.0mm -> DM50:XTAL_ABS05-32.768KHZ-9-T
- moved J4 6.10 mm to (134.9, 104.7), turned to -90 degrees
- moved R13 4.25 mm to (136.2, 95.0)
- moved R3 3.75 mm to (126.2, 101.2), turned to 0 degrees
- moved U6 2.34 mm to (117.8, 86.2)
- moved R12 2.16 mm to (120.1, 83.8)
- moved C23 2.12 mm to (114.8, 86.2)
- moved C22 2.11 mm to (121.0, 86.2)
- moved U4 0.42 mm to (126.5, 83.5)
- moved D3 0.10 mm to (133.6, 116.3)
Connections:
- BT1 pad 1: VBAT -> Net-(BT1-+)
- C23 pad 1: VBAT -> Net-(D4-A)
- D2 pad 1: VBAT -> Net-(BT1-+)
- J4 pad 1: VBAT -> GND
- J4 pad 2: GND -> Net-(D4-A)
- U2 pad 1: VBAT -> 3.3V
- U6 pad 3: VBAT -> Net-(D4-A)
- U6 pad 4: VBUS -> Net-(JP1-A)
Routing:
- net VBAT: track 53.0 -> 0.00 mm, vias 2 -> 0
- net Net-(D4-A): track 0.00 -> 44.0 mm, vias 0 -> 2
- net Net-(BT1-+): track 0.00 -> 14.7 mm
- net Net-(JP1-A): track 0.00 -> 8.59 mm
- net Net-(D3-A): track 16.7 -> 23.0 mm
- net Net-(D1-A): track 14.4 -> 19.4 mm
- net Net-(D3-K): track 44.0 -> 48.9 mm
- net GND: track 170.7 -> 174.0 mm, vias 134 -> 138
- net VBUS: track 37.2 -> 34.0 mm
- net USB_DM (D-): track 16.2 -> 17.8 mm
- net Net-(J2-D--PadA7): track 8.47 -> 9.98 mm
- net USB_DP (D+): track 16.5 -> 17.2 mm
- net 3.3V: track 176.7 -> 177.3 mm
- net Net-(U6-PROG): track 1.07 -> 1.62 mm
Other:
- board text added: "LiPO"
- board text added: "ON"
- board text added: "charging"
- board text removed: "+ LiPO (optional)"
- board text removed: "- LiPO (optional)"

Commit message: pcb changes
Routing:
- net ROW09/WAKEUP: track 160.5 -> 162.7 mm
- net ROW03: track 90.0 -> 91.7 mm
- net ROW07: track 132.9 -> 133.5 mm
- net GND: vias 138 -> 137
Other:
- outline, holes or cut-outs redrawn
- board text added: "(easy) Programming via USB (Bootloader mode) ------------------------------------- 1. Connect PCB to your computer via USB. 2. Press and hold PGM button. 3. Press and release the RESET button. 4. Release the PGM button. This action activates the bootloader. 5. Open your preferred STM32 bootloader software . (e.g., STM32CubeProgrammer). 6. Load firmware file. 7. Programming the Microcontroller. (d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"
- board text added: "+"
- board text added: "-"
- board text added: "28 x 22"
- board text added: "9 x 37"
- board text added: "JST PH 2.0mm"
- board text added: "LiPO 3.7V"
- board text added: "LiPO ZONE A"
- board text added: "LiPO ZONE B"
- board text added: "MAX H=4mm"
- board text added: "mods: 302025, 302323, 401525, 402020, 402025"
- board text removed: "(easy) Programming via USB (Bootloader mode) ------------------------------------- 1. Connect PCB to your computer via USB. 2. Press and hold PGM button. 3. Press and release the RESET button . 4. Release the PGM button. This action activates the bootloader. 5. Open your preferred STM32 bootloader software . (e.g., STM32CubeProgrammer). 6. Load firmware file. 7. Programming the Microcontroller. (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"

Commit message: pcb changes
Parts:
- moved C22 2.73 mm to (122.2, 83.8), turned to 0 degrees
- moved JP1 1.11 mm to (122.2, 86.2), turned to 0 degrees
- moved J4 1.04 mm to (134.6, 103.7)
- moved R12 0.85 mm to (119.2, 83.8)
Routing:
- net Net-(JP1-A): track 8.59 -> 2.98 mm
- net GND: track 174.0 -> 172.1 mm, vias 137 -> 245
- net COL06: track 85.7 -> 84.6 mm
- net Net-(D3-K): track 48.9 -> 50.1 mm
- net Net-(D1-A): track 19.4 -> 20.4 mm
- net Net-(D4-A): track 44.0 -> 43.3 mm, vias 2 -> 3
- net USB_DM (D-): track 17.8 -> 18.3 mm
