File: hardware/DM50.kicad_pcb (KiCad board)
At the start: 2 copper layers, 70 x 151 mm, 112 parts, among them J1 ST-LINK, J2 USB_C_Receptacle_USB2.0_14P, J3 SERIAL, J4 LiPO 3,7V, Q1 MMBT3904, SW1 SW_SPST, SW10 BT_SMD, SW11 BT_SMD, SW12 BT_SMD, SW13 BT_SMD, SW14 BT_SMD, SW15 BT_SMD, SW16 BT_SMD, SW17 BT_SMD, SW18 BT_SMD, SW19 BT_SMD, SW2 BT_SMD, SW20 BT_SMD, SW21 BT_SMD, SW22 BT_SMD, SW23 BT_SMD, SW24 BT_SMD, SW25 BT_SMD, SW26 BT_SMD, SW27 BT_SMD, SW28 BT_SMD, SW29 BT_SMD, SW3 BT_SMD, SW30 BT_SMD, SW31 BT_SMD, SW32 BT_SMD, SW33 BT_SMD, SW34 BT_SMD, SW35 BT_SMD, SW36 BT_SMD, SW37 BT_SMD, SW38 BT_SMD, SW39 BT_SMD, SW4 BT_SMD, SW40 BT_SMD, SW41 BT_SMD, SW42 SW_SPST, SW43 BT_SMD, SW44 BT_SMD, SW45 BT_SMD, SW46 BT_SMD, SW47 BT_SMD, SW48 BT_SMD, SW49 BT_SMD, SW5 BT_SMD, SW50 BT_SMD, SW51 BT_SMD, SW52 BT_SMD, SW6 BT_SMD, SW7 BT_SMD, SW8 BT_SMD, SW9 BT_SMD, U1 EA_DOGL128X-6, U2 STM32U575RIT6, U3 W25Q128JVSIQ, U4 USBLC6-2SC6, U5 ADP2108AUJ-3.3, U6 MCP73831, Y1 32768

Commit message: Update DM50.kicad_pcb
Parts:
- moved C16 24.3 mm to (106.1, 93.5), turned to -90 degrees
- moved C18 21.0 mm to (98.8, 87.8), turned to 90 degrees
- moved BZ1 10.8 mm to (112.8, 72.2), turned to 0 degrees
- moved C15 5.52 mm to (111.1, 69.8), turned to 0 degrees
- moved R7 4.01 mm to (113.3, 74.8), turned to 0 degrees
- moved R4 2.05 mm to (116.6, 101.5), turned to -90 degrees
- moved U3 1.90 mm to (100.0, 94.9)
- moved C21 1.53 mm to (104.3, 93.5), turned to -90 degrees
- moved Q1 1.25 mm to (116.6, 77.0)
- moved C20 1.05 mm to (118.1, 101.5), turned to 90 degrees
- moved R12 0.69 mm to (128.1, 104.5)
Routing:
- net GND: track 410.8 -> 442.3 mm, vias 147 -> 151
- net VBUS: track 36.9 -> 44.0 mm
- net SWD_SWDIO: track 16.6 -> 22.6 mm
- net VINPUT: track 12.7 -> 18.4 mm
- net VBAT_SNS: track 47.1 -> 52.8 mm
- net COL06: track 88.4 -> 93.6 mm
- net 3.3V: track 239.1 -> 244.2 mm
- net COL03: track 120.1 -> 124.0 mm
- net Net-(U1-CAP3P): track 3.28 -> 6.52 mm
- net Net-(U1-V3): track 2.83 -> 6.06 mm
- net Net-(U1-V0): track 2.85 -> 6.07 mm
- net Net-(U1-CAP1P): track 2.86 -> 6.07 mm
- net Net-(U1-V2): track 2.87 -> 6.08 mm
- net Net-(U1-V4): track 2.89 -> 6.09 mm
- net Net-(U1-V1): track 2.91 -> 6.11 mm
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Other:
- outline, holes or cut-outs redrawn

Commit message: pcb updates
Parts:
- removed U1: EA_DOGL128X-6, DM50:EA_DOGL128-6
- added C25: 1uF, Capacitor_SMD:C_0603_1608Metric, F.Cu at (91.6, 31.8)
- added J5: Micro_SD_Card, Connector_Card:microSD_HC_Hirose_DM3AT-SF-PEJM5, F.Cu at (80.4, 33.2)
- added R16: 10K, Resistor_SMD:R_0603_1608Metric, F.Cu at (90.7, 38.5)
- added R17: 10K, Resistor_SMD:R_0603_1608Metric, F.Cu at (90.8, 36.0)
- added R18: 10K, Resistor_SMD:R_0603_1608Metric, F.Cu at (91.6, 33.8)
- added R19: 10K, Resistor_SMD:R_0603_1608Metric, F.Cu at (91.6, 29.8)
- added R20: 10K, Resistor_SMD:R_0603_1608Metric, F.Cu at (91.6, 28.2)
- C11, C13: value 9pF -> 6pF
- U2: value STM32U575RIT6 -> STM32U595RJTx
- moved J3 78.9 mm to (155.9, 82.1), turned to 90 degrees
- moved R8 51.7 mm to (135.5, 32.8)
- moved C13 51.5 mm to (100.7, 26.2)
- moved C14 50.1 mm to (115.8, 36.2), turned to -90 degrees
- moved C11 49.6 mm to (101.8, 25.1)
- moved Y1 49.4 mm to (102.8, 27.2)
- moved U2 49.3 mm to (106.8, 35.0)
- moved BZ1 49.2 mm to (143.1, 33.5)
- moved C17 49.1 mm to (106.8, 26.2), turned to 0 degrees
- moved U3 48.2 mm to (99.6, 46.7), turned to -90 degrees
- moved C16 47.8 mm to (108.1, 45.8)
- moved C21 47.8 mm to (106.3, 45.8)
- moved Q1 45.1 mm to (136.8, 36.7)
- moved R7 40.6 mm to (137.3, 42.0)
- moved C18 40.0 mm to (85.1, 50.2)
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Connections:
- R5 pad 1: ROW09/WAKEUP -> GND
- R5 pad 2: GND -> ROW09
- SW48 pad 2: ROW09/WAKEUP -> ROW09
- SW49 pad 2: ROW09/WAKEUP -> ROW09
- SW50 pad 2: ROW09/WAKEUP -> ROW09
- SW51 pad 2: ROW09/WAKEUP -> ROW09
- SW52 pad 2: ROW09/WAKEUP -> ROW09
- U2 pad 10: VBAT_SNS -> ROW06
- U2 pad 11: CHARG_SNS -> ROW07
- U2 pad 14: QUADSPI_NCS -> ROW08
- U2 pad 15: COL01 -> ROW09
- U2 pad 16: USART_TX -> QUADSPI_NCS
- U2 pad 17: USART_RX -> unconnected-(U2-PA3-Pad17)
- U2 pad 2: unconnected-(U2-PC13-Pad2) -> ROW01
- U2 pad 20: unconnected-(U2-PA4-Pad20) -> DAC1_OUT1
- U2 pad 21: unconnected-(U2-PA5-Pad21) -> DAC1_OUT2
- U2 pad 24: ROW01 -> ADC_IN
- U2 pad 25: COL02 -> VBAT_SNS
- U2 pad 28: ROW02 -> CHARG_SNS
- U2 pad 33: COL03 -> COL01
- U2 pad 34: ROW03 -> COL02
- U2 pad 35: COL04 -> COL03
- U2 pad 36: ROW04 -> COL04
- U2 pad 38: ROW05 -> COL06
- U2 pad 39: COL06 -> SD_D0
- U2 pad 40: ROW06 -> SD_D1
- U2 pad 41: ROW07 -> LED
- U2 pad 42: ROW08 -> USART_TX
- U2 pad 43: unconnected-(U2-PA10-Pad43) -> USART_RX
- U2 pad 5: unconnected-(U2-PH0-Pad5) -> ROW02
- U2 pad 50: unconnected-(U2-PA15-Pad50) -> SWD_JTDI
- U2 pad 51: ROW09/WAKEUP -> SD_D2
- U2 pad 52: BUZZER -> SD_D3
- U2 pad 53: unconnected-(U2-PC12-Pad53) -> SD_CK
- U2 pad 54: unconnected-(U2-PD2-Pad54) -> SD_CMD
- U2 pad 56: unconnected-(U2-PB4-Pad56) -> SWD_JTRST
- U2 pad 6: unconnected-(U2-PH1-Pad6) -> ROW03
- U2 pad 8: ADC_IN -> ROW04
- U2 pad 9: unconnected-(U2-PC1-Pad9) -> ROW05
Routing:
- net GND: track 442.3 -> 258.4 mm, vias 151 -> 141
- net ROW09/WAKEUP: track 159.5 -> 0.00 mm, vias 2 -> 0
- net 3.3V: track 244.2 -> 84.9 mm, vias 3 -> 5
- net ROW09: track 0.00 -> 153.6 mm, vias 0 -> 1
- net NRST: track 82.1 -> 16.4 mm, vias 2 -> 1
- net Net-(BT1--): track 69.6 -> 7.62 mm
- net BOOT0: track 63.9 -> 12.4 mm, vias 2 -> 1
- net SD_D2: track 0.00 -> 51.5 mm, vias 0 -> 2
- net SD_D3: track 0.00 -> 46.5 mm, vias 0 -> 2
- net SD_CMD: track 0.00 -> 44.9 mm, vias 0 -> 2
- net CHARG_SNS: track 50.2 -> 7.74 mm
- net COL01: track 138.9 -> 97.8 mm, vias 3 -> 0
- net VBAT_SNS: track 52.8 -> 12.2 mm
- net SD_D1: track 0.00 -> 37.7 mm, vias 0 -> 2
- net SD_D0: track 0.00 -> 37.3 mm, vias 0 -> 2
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
Commit message: pcb changes
Parts:
- removed J1: ST-LINK, DM50:SAMTEC-SMH-105-02-X-S
- removed J3: SERIAL, DM50:SAMTEC-SMH-105-02-X-S
- added J6: DEBUG, SERIAL, DM50:610110249221, F.Cu at (136.3, 82.2)
- added U1: EA_DOGL128X-6, DM50:EA_DOGL128-6, F.Cu at (82.2, 112.2)
- J5: footprint Connector_Card:microSD_HC_Hirose_DM3AT-SF-PEJM5 -> DM50:SAMTEC-SMH-105-02-X-S
- moved C25 49.1 mm to (91.2, 80.9)
- moved R16 49.1 mm to (90.3, 87.6)
- moved R17 49.1 mm to (90.5, 85.1)
- moved R18 49.1 mm to (91.2, 82.9)
- moved R19 49.1 mm to (91.2, 78.9)
- moved R20 49.1 mm to (91.2, 77.4)
- moved J5 49.1 mm to (76.5, 82.2)
- moved C12 47.3 mm to (102.1, 87.7)
- moved C14 47.3 mm to (119.6, 83.4)
- moved C16 47.3 mm to (111.8, 92.9)
- moved C17 47.3 mm to (110.6, 73.4)
- moved C21 47.3 mm to (110.1, 92.9)
- moved C24 47.3 mm to (106.8, 92.9)
- moved R15 47.3 mm to (108.3, 92.9)
- moved R5 47.3 mm to (99.8, 99.4)
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Routing:
- net GND: track 258.4 -> 279.7 mm, vias 141 -> 132
- net 3.3V: track 84.9 -> 69.9 mm, vias 5 -> 4
- net USB_DM (D-): track 32.0 -> 20.1 mm
- net USB_DP (D+): track 35.9 -> 24.9 mm
- net DISP_SI: track 25.0 -> 33.9 mm
- net DISP_SCL: track 27.2 -> 35.4 mm
- net DISP_A0: track 29.6 -> 37.4 mm
- net Net-(BT1--): track 7.62 -> 0.00 mm
- net DISP_RST: track 30.1 -> 37.2 mm
- net DISP_CS1B: track 32.8 -> 39.0 mm
- net ROW07: track 136.9 -> 131.9 mm
- net Net-(BT1-+): track 14.0 -> 9.30 mm
- net SD_D0: track 37.3 -> 41.7 mm
- net SD_D1: track 37.7 -> 41.8 mm
- net SD_CK: track 35.5 -> 39.1 mm
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
Commit message: pcb upgrades
Parts:
- removed BZ1: Buzzer, DM50:Buzzer
- removed Q1: MMBT3904, Package_TO_SOT_SMD:SOT-23
- added J1: SJ2-35954D-SMT-TR, DM50:CUI_SJ2-35954D-SMT-TR, F.Cu at (77.3, 104.2)
- added J3: Speaker, DM50:Buzzer, F.Cu at (90.2, 98.8)
- added U7: TPA6111A2DR, Package_SO:SOIC-8-1EP_3.9x4.9mm_P1.27mm_EP2.41x3.81mm_ThermalVias, F.Cu at (88.4, 104.5)
- J5: footprint DM50:SAMTEC-SMH-105-02-X-S -> DM50:502570-0893_MOL
- R7: value 100K -> 10K
- moved C15 81.0 mm to (97.8, 111.0)
- moved R7 81.0 mm to (98.3, 113.0)
- moved R8 81.0 mm to (96.5, 103.7)
- moved SW42 73.8 mm to (139.2, 70.8), turned to 90 degrees
- moved R2 67.6 mm to (135.2, 68.8), turned to 0 degrees
- moved C10 63.9 mm to (135.2, 72.8), turned to 180 degrees
- moved C18 59.7 mm to (91.5, 110.5), turned to 180 degrees
- moved C19 53.6 mm to (92.0, 104.5)
- moved R1 28.4 mm to (77.3, 72.8)
- moved SW1 26.2 mm to (73.5, 70.8)
- moved J5 3.20 mm to (79.7, 82.1), turned to 90 degrees
Connections:
- net CHARG renamed Net-(D3-K)
- R7 pad 1: 3.3V -> DAC1_OUT1
- R8 pad 1: BUZZER -> Net-(U7-IN2-)
- R8 pad 2: Net-(Q1-B) -> DAC1_OUT2
- U2 pad 17: unconnected-(U2-PA3-Pad17) -> AUDIO_ONOFF
Routing:
- net GND: track 279.7 -> 253.4 mm
- net Net-(U7-VO1): track 0.00 -> 18.7 mm
- net Net-(U7-VO2): track 0.00 -> 16.9 mm
- net NRST: track 16.4 -> 7.16 mm
- net BOOT0: track 12.4 -> 4.13 mm
- net Net-(J3-Pin_1): track 0.00 -> 6.24 mm
- net 3.3V: track 69.9 -> 65.1 mm
- net SD_D2: track 54.3 -> 52.9 mm
- net SD_CMD: track 45.1 -> 43.7 mm
Other:
- outline, holes or cut-outs redrawn

Commit message: pcb changes
Parts:
- removed J1: SJ2-35954D-SMT-TR, DM50:CUI_SJ2-35954D-SMT-TR
- added C26: 100nF, Capacitor_SMD:C_1206_3216Metric, F.Cu at (111.3, 101.8)
- added C27: 68µF, Capacitor_SMD:C_1210_3225Metric, F.Cu at (90.2, 109.0)
- added C28: 68µF, Capacitor_SMD:C_1210_3225Metric, F.Cu at (80.8, 109.0)
- added C29: 1µF, Capacitor_SMD:C_1206_3216Metric, F.Cu at (93.8, 98.0)
- added J7: SJ-43516-SMT-TR, DM50:SJ-43516-SMT_CUD, F.Cu at (80.8, 102.3)
- added R21: 20K, Resistor_SMD:R_0603_1608Metric, F.Cu at (97.8, 98.8)
- added R22: 20K, Resistor_SMD:R_0603_1608Metric, F.Cu at (95.5, 108.5)
- R7, R8: value 10K -> 20K
- moved R7 15.8 mm to (97.8, 97.2), turned to 180 degrees
- moved C18 11.7 mm to (102.8, 107.2), turned to 0 degrees
- moved C19 10.8 mm to (102.8, 103.8), turned to 0 degrees
- moved C15 7.29 mm to (102.8, 105.5)
- moved U7 7.21 mm to (95.5, 103.7)
- moved R8 6.52 mm to (95.5, 110.2)
- moved R5 4.13 mm to (104.0, 99.2), turned to 0 degrees
- moved J3 3.86 mm to (86.5, 97.3), turned to 180 degrees
Connections:
- U7 pad 3: unconnected-(U7-BYPASS-Pad3) -> Net-(U7-BYPASS)
Routing:
- net Net-(U7-VO1): track 18.7 -> 0.00 mm
- net Net-(U7-VO2): track 16.9 -> 0.00 mm
- net Net-(J3-Pin_1): track 6.24 -> 0.00 mm
- net 3.3V: track 65.1 -> 62.1 mm

Commit message: pcb upgrade
Parts:
- removed C21: 2.2uF, Capacitor_SMD:C_0603_1608Metric
- added C30: 68µF, Capacitor_SMD:C_1210_3225Metric, F.Cu at (109.5, 96.2)
- moved C28 19.8 mm to (100.5, 109.3), turned to 180 degrees
- moved C27 11.6 mm to (100.5, 103.8), turned to 90 degrees
- moved L1 6.30 mm to (118.3, 97.5), turned to 180 degrees
- moved R14 5.51 mm to (125.3, 101.5)
- moved C18 5.23 mm to (108.0, 107.0)
- moved R19 4.62 mm to (95.8, 79.2)
- moved R20 4.62 mm to (95.8, 77.8)
- moved R2 4.10 mm to (135.3, 72.8)
- moved R12 4.01 mm to (125.3, 103.2), turned to 0 degrees
- moved C19 3.94 mm to (106.2, 101.8)
- moved C10 3.91 mm to (135.3, 68.8)
- moved C15 3.71 mm to (106.4, 104.8)
- moved C26 3.35 mm to (114.5, 100.8)
- moved U4 2.50 mm to (129.3, 100.0), turned to 90 degrees
- moved R18 1.94 mm to (89.8, 84.2)
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Connections:
- J6 pad 1: 3.3V -> USART_TX
- J6 pad 10: SWD_SWO -> SWD_SWCLK
- J6 pad 2: USART_TX -> USART_RX
- J6 pad 3: USART_RX -> ADC_IN
- J6 pad 4: ADC_IN -> SWD_SWDIO
- J6 pad 7: SWD_SWDIO -> NRST
- J6 pad 8: SWD_SWCLK -> 3.3V
- J6 pad 9: NRST -> SWD_SWO
- U2 pad 30: VCAP1 -> Net-(U2-VCAP)
- U2 pad 50: SWD_JTDI -> unconnected-(U2-PA15-Pad50)
- U2 pad 56: SWD_JTRST -> unconnected-(U2-PB4-Pad56)
Routing:
- net 3.3V: track 62.1 -> 200.6 mm
- net Net-(BT1--): track 0.00 -> 70.4 mm
- net NRST: track 7.16 -> 60.8 mm, vias 1 -> 2
- net Net-(C28-Pad1): track 0.00 -> 44.6 mm
- net GND: track 253.4 -> 290.7 mm
- net AUDIO_ONOFF: track 0.00 -> 31.1 mm, vias 0 -> 2
- net Net-(C27-Pad1): track 0.00 -> 23.5 mm
- net ROW09: track 153.6 -> 135.9 mm
- net Net-(D3-K): track 5.16 -> 21.7 mm
- net SD_D2: track 52.9 -> 66.7 mm
- net SD_D1: track 41.8 -> 54.9 mm
- net SD_D3: track 49.3 -> 61.8 mm
- net ROW07: track 131.9 -> 119.4 mm
- net SD_CMD: track 43.7 -> 56.0 mm
- net USART_TX: track 3.61 -> 15.8 mm, vias 1 -> 0
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Other:
- board text added: "SPEAKER"
- board text removed: "-"
- board text removed: "BUZZER"

Commit message: pcb upgrades
Parts:
- moved C18 35.3 mm to (110.5, 71.8)
- moved R5 8.53 mm to (112.1, 101.5), turned to -90 degrees
- moved J7 2.90 mm to (80.9, 105.2)
- moved C25 2.85 mm to (92.3, 81.8), turned to 180 degrees
- moved JP1 2.47 mm to (127.3, 108.8)
- moved J3 2.22 mm to (86.2, 99.5)
- turned R1 to 0 degrees
Connections:
- U2 pad 10: ROW06 -> ROW03
- U2 pad 11: ROW07 -> ROW04
- U2 pad 14: ROW08 -> COL03
- U2 pad 15: ROW09 -> ROW05
- U2 pad 2: ROW01 -> LED
- U2 pad 33: COL01 -> ROW06
- U2 pad 34: COL02 -> ROW07
- U2 pad 35: COL03 -> COL04
- U2 pad 36: COL04 -> ROW08
- U2 pad 37: COL05 -> ROW09
- U2 pad 38: COL06 -> COL05
- U2 pad 41: LED -> COL06
- U2 pad 5: ROW02 -> COL01
- U2 pad 6: ROW03 -> ROW01
- U2 pad 8: ROW04 -> ROW02
- U2 pad 9: ROW05 -> COL02
Routing:
- net ROW01: track 19.6 -> 84.8 mm, vias 1 -> 2
- net 3.3V: track 200.6 -> 254.1 mm, vias 4 -> 2
- net COL01: track 95.6 -> 148.5 mm, vias 0 -> 1
- net COL02: track 94.2 -> 140.3 mm, vias 0 -> 1
- net GND: track 290.7 -> 334.2 mm, vias 132 -> 138
- net BOOT0: track 14.3 -> 57.7 mm, vias 1 -> 2
- net ROW02: track 50.0 -> 93.2 mm, vias 3 -> 2
- net DAC1_OUT2: track 2.73 -> 45.8 mm, vias 1 -> 2
- net COL03: track 98.6 -> 133.7 mm, vias 0 -> 1
- net COL06: track 62.6 -> 95.1 mm, vias 1 -> 2
- net VBAT_SNS: track 11.1 -> 41.9 mm
- net ROW03: track 62.0 -> 92.1 mm, vias 2 -> 3
- net ROW04: track 72.3 -> 99.9 mm, vias 2 -> 4
- net COL05: track 103.8 -> 129.7 mm, vias 0 -> 1
- net COL04: track 100.5 -> 124.7 mm, vias 0 -> 1
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
Commit message: update images
Parts:
- moved C26 5.22 mm to (109.3, 101.2)
- moved L1 4.53 mm to (114.6, 100.0), turned to 90 degrees
- moved C15 4.37 mm to (105.3, 100.5), turned to -90 degrees
- moved R5 1.75 mm to (112.1, 103.2), turned to 90 degrees
- moved C19 1.57 mm to (107.1, 100.5), turned to -90 degrees
- moved C28 0.85 mm to (100.5, 108.5)
Routing:
- net GND: track 334.2 -> 351.9 mm, vias 138 -> 153
- net 3.3V: track 254.1 -> 244.6 mm
- net DAC1_OUT1: track 18.4 -> 22.5 mm
- net Net-(C28-Pad1): track 41.6 -> 39.3 mm
- net Net-(U5-SW): track 4.66 -> 2.48 mm
- net Net-(C27-Pad1): track 22.7 -> 22.1 mm
- net Net-(D3-A): track 4.56 -> 5.06 mm
- net Net-(D1-A): track 12.7 -> 13.2 mm
